Commit message: add data

File: legged_gym/assets/www_box/www_box.urdf (robot description, URDF)
Before this commit: robot largebox, 1 links, 0 joints
Links:
- link largebox_link: mass 0.1 -> 5.0; geometry collision mesh filename=www_box.obj scale=1.0 1.0 1.0; visual mesh filename=www_box.obj scale=1.0 1.0 1.0
