Commit message: virtual curriculum update

File: legged_gym/assets/box/box.urdf (robot description, URDF)
Before this commit: robot box, 1 links, 0 joints
Links:
- link box_link: mass 4.0 -> 0.1

File: legged_gym/assets/www_box/www_box.urdf (robot description, URDF)
Before this commit: robot largebox, 1 links, 0 joints
Links:
- link largebox_link: mass 5.0 -> 4.0
